File: OttoWah/OttoWah.sch (KiCad schematic (older format))
At the start: 20 parts, among them J1 Conn_01x01_Female, J2 Conn_01x01_Female, J3 Conn_01x01_Female, J4 Conn_01x01_Female, J5 Conn_01x01_Female, U1 TL072, U2 Optocoupler

Commit message: Updated schematic
- Added decoupling caps to power rails
- Added power and effect on indicators
- Began assigning footprints
Parts:
- removed J1, J2: Conn_01x01_Female, symbol Connector:Conn_01x01_Female
- added C5, C6: 10uF, symbol Device:C
- added D1, D2: LED, symbol Device:LED
- added J1, J2: Conn_01x02_Female, Connector_PinHeader_2.54mm:PinHeader_1x02_P2.54mm_Vertical, symbol Connector:Conn_01x02_Female
- added J6: Conn_01x01_Female, Connector_PinHeader_2.54mm:PinHeader_1x01_P2.54mm_Vertical, symbol Connector:Conn_01x01_Female
- added R8, R9: 1k, symbol Device:R_US
- J3, J4, J5: footprint (none) -> Connector_PinHeader_2.54mm:PinHeader_1x01_P2.54mm_Vertical
- U1: footprint (none) -> Package_DIP:DIP-8_W7.62mm_Socket
- U1: renamed from U?; footprint (none) -> Package_DIP:DIP-8_W7.62mm_Socket
Connections:
- net +9V: now also C6.2, R8.2
- net -9V: now also C5.1
- net GND: now also C5.2, C6.1, D1.1 (K), D2.1 (K), J1.2 (Pin_2), J2.2 (Pin_2)
- net at C1.2: now also J1.1 (Pin_1)
- net at RV2.2: now also J2.1 (Pin_1)
- new net: D1.2 (A), R8.1
- new net: D2.2 (A), R9.1
- new net: J6.1 (Pin_1), R9.2
Other:
- note added: "EFFECT ON IND.\n"
- note added: "POWER ON IND.\n"
- moved on the sheet: U1C

Commit message: Finished preliminary layout and routing.
Parts:
- C1, C2, C3, C4, C5, C6: footprint (none) -> Capacitor_THT:C_Disc_D5.0mm_W2.5mm_P5.00mm
- D1, D2: footprint (none) -> LED_THT:LED_D5.0mm
- R1, R2, R3, R5, R6, R7, R8, R9: footprint (none) -> Resistor_THT:R_Axial_DIN0204_L3.6mm_D1.6mm_P5.08mm_Horizontal
- RV1, RV2: footprint (none) -> Connector_PinHeader_2.54mm:PinHeader_1x03_P2.54mm_Vertical
- U2: footprint (none) -> ElectronicsForGuitarists-DentonDaily:Optocoupler
Changed lines of the file:
@@
 F 0 "C1" V 3048 4550 50  0000 C CNN
 F 1 "0.1uF" V 3139 4550 50  0000 C CNN
-F 2 "" H 3338 4400 50  0001 C CNN
+F 2 "Capacitor_THT:C_Disc_D5.0mm_W2.5mm_P5.00mm" H 3338 4400 50  0001 C CNN
 F 3 "~" H 3300 4550 50  0001 C CNN
 	1    3300 4550
@@
 F 0 "R1" H 3618 4846 50  0000 L CNN
 F 1 "100k" H 3618 4755 50  0000 L CNN
-F 2 "" V 3590 4790 50  0001 C CNN
+F 2 "Resistor_THT:R_Axial_DIN0204_L3.6mm_D1.6mm_P5.08mm_Horizontal" V 3590 4790 50  0001 C CNN
 F 3 "~" H 3550 4800 50  0001 C CNN
 	1    3550 4800
@@
 F 0 "RV1" V 4495 3600 50  0000 C CNN
 F 1 "25k_LIN" V 4586 3600 50  0000 C CNN
-F 2 "" H 4700 3600 50  0001 C CNN
+F 2 "Connector_PinHeader_2.54mm:PinHeader_1x03_P2.54mm_Vertical" H 4700 3600 50  0001 C CNN
 F 3 "~" H 4700 3600 50  0001 C CNN
 	1    4700 3600
@@
 F 0 "R3" V 3795 2950 50  0000 C CNN
 F 1 "100k" V 3886 2950 50  0000 C CNN
-F 2 "" V 4040 2940 50  0001 C CNN
+F 2 "Resistor_THT:R_Axial_DIN0204_L3.6mm_D1.6mm_P5.08mm_Horizontal" V 4040 2940 50  0001 C CNN
 F 3 "~" H 4000 2950 50  0001 C CNN
 	1    4000 2950
@@
 F 0 "R2" V 2995 2950 50  0000 C CNN
 F 1 "2.2k" V 3086 2950 50  0000 C CNN
-F 2 "" V 3240 2940 50  0001 C CNN
+F 2 "Resistor_THT:R_Axial_DIN0204_L3.6mm_D1.6mm_P5.08mm_Horizontal" V 3240 2940 50  0001 C CNN
 F 3 "~" H 3200 2950 50  0001 C CNN
 	1    3200 2950
@@
 F 0 "R5" V 4945 3600 50  0000 C CNN
 F 1 "1k" V 5036 3600 50  0000 C CNN
-F 2 "" V 5190 3590 50  0001 C CNN
+F 2 "Resistor_THT:R_Axial_DIN0204_L3.6mm_D1.6mm_P5.08mm_Horizontal" V 5190 3590 50  0001 C CNN
 F 3 "~" H 5150 3600 50  0001 C CNN
 	1    5150 3600
@@
 Wire Wire Line
 	5300 3600 5400 3600
-Wire Wire Line
-	5400 3600 5400 3700
-Wire Wire Line
-	5600 3700 5600 3600
-Wire Wire Line
-	5400 4000 5400 4100
-Wire Wire Line
-	5600 4000 5600 4100
 $Comp
 L power:GND #PWR0103
@@
 F 0 "R6" V 5795 4550 50  0000 C CNN
 F 1 "120k" V 5886 4550 50  0000 C CNN
-F 2 "" V 6040 4540 50  0001 C CNN
+F 2 "Resistor_THT:R_Axial_DIN0204_L3.6mm_D1.6mm_P5.08mm_Horizontal" V 6040 4540 50  0001 C CNN
 F 3 "~" H 6000 4550 50  0001 C CNN
 	1    6000 4550
@@
 F 0 "C2" V 6248 4550 50  0000 C CNN
 F 1 "0.01uF" V 6339 4550 50  0000 C CNN
-F 2 "" H 6538 4400 50  0001 C CNN
+F 2 "Capacitor_THT:C_Disc_D5.0mm_W2.5mm_P5.00mm" H 6538 4400 50  0001 C CNN
 F 3 "~" H 6500 4550 50  0001 C CNN
 	1    6500 4550
@@
 F 0 "C3" V 6898 3600 50  0000 C CNN
 F 1 "0.01uF" V 6989 3600 50  0000 C CNN
-F 2 "" H 7188 3450 50  0001 C CNN
+F 2 "Capacitor_THT:C_Disc_D5.0mm_W2.5mm_P5.00mm" H 7188 3450 50  0001 C CNN
 F 3 "~" H 7150 3600 50  0001 C CNN
 	1    7150 3600
@@
 F 0 "R7" V 6945 4050 50  0000 C CNN
 F 1 "270k" V 7036 4050 50  0000 C CNN
-F 2 "" V 7190 4040 50  0001 C CNN
+F 2 "Resistor_THT:R_Axial_DIN0204_L3.6mm_D1.6mm_P5.08mm_Horizontal" V 7190 4040 50  0001 C CNN
 F 3 "~" H 7150 4050 50  0001 C CNN
 	1    7150 4050
@@
 Wire Wire Line
 	3550 4550 3550 3700
-$Comp
-L ElectronicsForGuitarists-DentonDaily:Optocoupler U2
-U 1 1 606C7113
-P 5500 3600
-F 0 "U2" H 5687 3389 50  0000 L CNN
-F 1 "Optocoupler" H 5687 3298 50  0000 L CNN
-F 2 "" H 5200 3650 50  0001 C CNN
-F 3 "" H 5200 3650 50  0001 C CNN
-	1    5500 3600
-	1    0    0    -1
-$EndComp
 Wire Wire Line
 	7000 4050 6750 4050
@@
 F 0 "C4" V 8155 4650 50  0000 C CNN
 F 1 "47uF" V 8064 4650 50  0000 C CNN
-F 2 "" H 7938 4500 50  0001 C CNN
+F 2 "Capacitor_THT:C_Disc_D5.0mm_W2.5mm_P5.00mm" H 7938 4500 50  0001 C CNN
 F 3 "~" H 7900 4650 50  0001 C CNN
 	1    7900 4650
@@
 F 0 "RV2" H 8083 4946 50  0000 R CNN
 F 1 "10k_LOG" H 8083 4855 50  0000 R CNN
-F 2 "" H 8150 4900 50  0001 C CNN
+F 2 "Connector_PinHeader_2.54mm:PinHeader_1x03_P2.54mm_Vertical" H 8150 4900 50  0001 C CNN
 F 3 "~" H 8150 4900 50  0001 C CNN
 	1    8150 4900
@@
 F 0 "C5" V 1398 1850 50  0000 C CNN
 F 1 "10uF" V 1489 1850 50  0000 C CNN
-F 2 "" H 1688 1700 50  0001 C CNN
+F 2 "Capacitor_THT:C_Disc_D5.0mm_W2.5mm_P5.00mm" H 1688 1700 50  0001 C CNN
 F 3 "~" H 1650 1850 50  0001 C CNN
 	1    1650 1850
@@
 F 0 "C6" V 1398 1550 50  0000 C CNN
 F 1 "10uF" V 1489 1550 50  0000 C CNN
-F 2 "" H 1688 1400 50  0001 C CNN
+F 2 "Capacitor_THT:C_Disc_D5.0mm_W2.5mm_P5.00mm" H 1688 1400 50  0001 C CNN
 F 3 "~" H 1650 1550 50  0001 C CNN
 	1    1650 1550
@@
 F 0 "D1" V 2839 1733 50  0000 R CNN
 F 1 "LED" V 2748 1733 50  0000 R CNN
-F 2 "" H 2800 1850 50  0001 C CNN
+F 2 "LED_THT:LED_D5.0mm" H 2800 1850 50  0001 C CNN
 F 3 "~" H 2800 1850 50  0001 C CNN
 	1    2800 1850
@@
 F 0 "D2" V 3639 1733 50  0000 R CNN
 F 1 "LED" V 3548 1733 50  0000 R CNN
-F 2 "" H 3600 1850 50  0001 C CNN
+F 2 "LED_THT:LED_D5.0mm" H 3600 1850 50  0001 C CNN
 F 3 "~" H 3600 1850 50  0001 C CNN
 	1    3600 1850
@@
 F 0 "R8" V 2595 1550 50  0000 C CNN
 F 1 "1k" V 2686 1550 50  0000 C CNN
-F 2 "" V 2840 1540 50  0001 C CNN
+F 2 "Resistor_THT:R_Axial_DIN0204_L3.6mm_D1.6mm_P5.08mm_Horizontal" V 2840 1540 50  0001 C CNN
 F 3 "~" H 2800 1550 50  0001 C CNN
 	1    2800 1550
@@
 F 0 "R9" V 3395 1550 50  0000 C CNN
 F 1 "1k" V 3486 1550 50  0000 C CNN
-F 2 "" V 3640 1540 50  0001 C CNN
+F 2 "Resistor_THT:R_Axial_DIN0204_L3.6mm_D1.6mm_P5.08mm_Horizontal" V 3640 1540 50  0001 C CNN
 F 3 "~" H 3600 1550 50  0001 C CNN
 	1    3600 1550
@@
 Text Notes 3300 1150 0    50   ~ 0
 EFFECT ON IND.\n
+$Comp
+L ElectronicsForGuitarists-DentonDaily:Optocoupler U2
+U 1 1 60671B34
+P 5500 3600
+F 0 "U2" H 5687 3389 50  0000 L CNN
+F 1 "Optocoupler" H 5687 3298 50  0000 L CNN
+F 2 "ElectronicsForGuitarists-DentonDaily:Optocoupler" H 5200 3650 50  0001 C CNN
+F 3 "" H 5200 3650 50  0001 C CNN
+	1    5500 3600
+	1    0    0    -1
+$EndComp
+Wire Wire Line
+	5400 3600 5400 3700
+Wire Wire Line
+	5600 3600 5600 3700
+Wire Wire Line
+	5400 4000 5400 4100
+Wire Wire Line
+	5600 4000 5600 4100
 $EndSCHEMATC

Commit message: Completely revamped layout and routing, and updated diode footprints. Should be ready for ordering!
Parts:
- D1, D2: footprint LED_THT:LED_D5.0mm -> Connector_PinHeader_2.54mm:PinHeader_1x02_P2.54mm_Vertical
Changed lines of the file:
@@
 F 0 "D1" V 2839 1733 50  0000 R CNN
 F 1 "LED" V 2748 1733 50  0000 R CNN
-F 2 "LED_THT:LED_D5.0mm" H 2800 1850 50  0001 C CNN
+F 2 "Connector_PinHeader_2.54mm:PinHeader_1x02_P2.54mm_Vertical" H 2800 1850 50  0001 C CNN
 F 3 "~" H 2800 1850 50  0001 C CNN
 	1    2800 1850
@@
 F 0 "D2" V 3639 1733 50  0000 R CNN
 F 1 "LED" V 3548 1733 50  0000 R CNN
-F 2 "LED_THT:LED_D5.0mm" H 3600 1850 50  0001 C CNN
+F 2 "Connector_PinHeader_2.54mm:PinHeader_1x02_P2.54mm_Vertical" H 3600 1850 50  0001 C CNN
 F 3 "~" H 3600 1850 50  0001 C CNN
 	1    3600 1850
